File: hardware/picow_ssr_control/manual_control.kicad_sch (KiCad schematic)
At the start: 1 part

Commit message: Power supply changes plus misc.
Parts:
- S1: Manufacturer_Name CTS -> (none); Manufacturer_Part_Number 193-8MS -> (none)
Changed lines of the file:
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@@
   (paper "USLetter")
   (title_block
-    (date "2023-01-28")
-    (rev "0.0.10")
+    (date "2023-02-08")
+    (rev "0.0.11")
     (comment 2 "http://creativecommons.org/licenses/by-sa/4.0/")
     (comment 3 "License: CC By SA 4.0")
@@
       (effects (font (size 1.27 1.27)) (justify left) hide)
     )
-    (property "Manufacturer_Name" "CTS" (id 12) (at 63.5 80.01 0)
-      (effects (font (size 1.27 1.27)) (justify left) hide)
-    )
-    (property "Manufacturer_Part_Number" "193-8MS" (id 13) (at 66.04 80.01 0)
-      (effects (font (size 1.27 1.27)) (justify left) hide)
-    )

Commit message: Pre KiCad 7.0.0 WIP
Parts:
- S1: Manufacturer_Name (none) -> CTS; Manufacturer_Part_Number (none) -> 193-8MS
Connections:
- net BANK_A.CNTL1 renamed BANK_A.OUT1
- net BANK_A.CNTL2 renamed BANK_A.OUT2
- net BANK_A.CNTL3 renamed BANK_A.OUT3
- net BANK_A.CNTL4 renamed BANK_A.OUT4
- net BANK_B.CNTL5 renamed BANK_B.OUT5
- net BANK_B.CNTL6 renamed BANK_B.OUT6
- net BANK_B.CNTL7 renamed BANK_B.OUT7
- net BANK_B.CNTL8 renamed BANK_B.OUT8
Changed lines of the file:
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@@
     (effects (font (size 1.27 1.27) bold) (justify left bottom))
   )
-  (label "BANK_B.CNTL8" (at 48.26 60.96 0)
+  (label "BANK_B.OUT8" (at 48.26 60.96 0)
     (effects (font (size 1.27 1.27)) (justify left bottom))
   )
-  (label "BANK_B.CNTL7" (at 48.26 58.42 0)
+  (label "BANK_B.OUT7" (at 48.26 58.42 0)
     (effects (font (size 1.27 1.27)) (justify left bottom))
   )
-  (label "BANK_B.CNTL6" (at 48.26 55.88 0)
+  (label "BANK_B.OUT6" (at 48.26 55.88 0)
     (effects (font (size 1.27 1.27)) (justify left bottom))
   )
-  (label "BANK_A.CNTL1" (at 48.26 43.18 0)
+  (label "BANK_A.OUT1" (at 48.26 43.18 0)
     (effects (font (size 1.27 1.27)) (justify left bottom))
   )
-  (label "BANK_A.CNTL3" (at 48.26 48.26 0)
+  (label "BANK_A.OUT3" (at 48.26 48.26 0)
     (effects (font (size 1.27 1.27)) (justify left bottom))
   )
-  (label "BANK_B.CNTL5" (at 48.26 53.34 0)
+  (label "BANK_B.OUT5" (at 48.26 53.34 0)
     (effects (font (size 1.27 1.27)) (justify left bottom))
   )
-  (label "BANK_A.CNTL2" (at 48.26 45.72 0)
+  (label "BANK_A.OUT2" (at 48.26 45.72 0)
     (effects (font (size 1.27 1.27)) (justify left bottom))
   )
-  (label "BANK_A.CNTL4" (at 48.26 50.8 0)
+  (label "BANK_A.OUT4" (at 48.26 50.8 0)
     (effects (font (size 1.27 1.27)) (justify left bottom))
   )
-  (hierarchical_label "BANK_A{CNTL[1..4]}" (shape passive) (at 76.2 38.1 0)
+  (hierarchical_label "BANK_A{OUT[1..4]}" (shape passive) (at 76.2 38.1 0)
     (effects (font (size 2 2) bold) (justify left))
   )
-  (hierarchical_label "BANK_B{CNTL[5..8]}" (shape passive) (at 76.2 66.04 0)
+  (hierarchical_label "BANK_B{OUT[5..8]}" (shape passive) (at 76.2 66.04 0)
     (effects (font (size 2 2) bold) (justify left))
   )
@@
       (effects (font (size 1.27 1.27)) (justify left) hide)
     )
+    (property "Manufacturer_Name" "CTS" (id 14) (at 44.45 22.86 0)
+      (effects (font (size 1.27 1.27)) (justify left) hide)
+    )
+    (property "Manufacturer_Part_Number" "193-8MS" (id 15) (at 44.45 20.32 0)
+      (effects (font (size 1.27 1.27)) (justify left) hide)
+    )

Commit message: Commit before trying changes to power system
Parts:
- S1: Height 9.37 -> (none); Manufacturer_Name CTS -> (none); Manufacturer_Part_Number 193-8MS -> (none)

Commit message: Commit before removing git submodule
Other:
- note added: "${SHEETNAME}"
- note removed: "Manual Control"
- company: (none) -> Michael Cummings
- title: (none) -> Pico W SSR Control
Changed lines of the file:
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@@
   (paper "USLetter")
   (title_block
-    (date "2023-02-13")
-    (rev "0.0.11")
-    (comment 2 "http://creativecommons.org/licenses/by-sa/4.0/")
-    (comment 3 "License: CC By SA 4.0")
-    (comment 4 "Author: Michael Cummings")
-    (comment 5 "https://ohwr.org/project/cernohl/wikis/Documents/CERN-OHL-version-2")
-    (comment 6 "Hardware License: CERN-OHL-W")
+    (title "Pico W SSR Control")
+    (date "2023-03-14")
+    (rev "0.0.12")
+    (company "Michael Cummings")
+    (comment 1 "https://ohwr.org/project/cernohl/wikis/Documents/CERN-OHL-version-2")
+    (comment 2 "Hardware License: CERN-OHL-W")
+    (comment 3 "https://creativecommons.org/licenses/by-sa/4.0/")
+    (comment 4 "License: CC By SA 4.0")
   )
   (junction (at 25.4 55.88) (diameter 0) (color 0 0 0 0)
@@
     (stroke (width 0) (type default))
   )
-  (text "Manual Control" (at 15.24 20.32 0)
+  (text "${SHEETNAME}" (at 15.24 20.32 0)
     (effects (font (size 4 4) bold) (justify left bottom))
   )
@@
   )
   (symbol (lib_id "power:GNDPWR") (at 25.4 66.04 0) (unit 1)
-    (in_bom yes) (on_board yes) (dnp no)
-    (property "Reference" "#PWR0101" (at 25.4 71.12 0)
+    (in_bom yes) (on_board yes) (dnp no) (fields_autoplaced)
+    (property "Reference" "#PWR015" (at 25.4 71.12 0)
       (effects (font (size 1.27 1.27)) hide)
     )
-    (property "Value" "GNDPWR" (at 25.4 69.596 0)
+    (property "Value" "GNDPWR" (at 25.273 71.12 0)
       (effects (font (size 1.27 1.27)))
     )
@@
       (project "picow_ssr_control"
         (path "/04b3a773-2568-4dd5-b3b9-f3130861ac39/6f32e7f5-0a22-4bb9-a836-1e48dd69b48f"
-          (reference "#PWR0101") (unit 1)
+          (reference "#PWR015") (unit 1)
         )
       )
