File: hardware/picow_ssr_control/picow_control.kicad_sch (KiCad schematic)
At the start: 17 parts, among them U1 RaspberryPi-PicoW

Commit message: Updated schemas
Parts:
- added C3: 100n, Capacitor_SMD:C_0805_2012Metric, symbol Device:C
- added Q2: DMG2305UX-7, Package_TO_SOT_SMD:SOT-23, symbol dragon_mobile:DMG2305UX-7
Connections:
- net GNDPWR: now also C3.2
- net VBUS: now also Q2.1 (G)
- net VSYS: now also C3.1, Q2.2 (S)
- new net +5V: Q2.3 (D)
Other:
- moved on the sheet: U1

Commit message: Power supply changes plus misc.
Parts:
- removed C3: 100n, Capacitor_SMD:C_0805_2012Metric, symbol Device:C
- added C11: 100n, Capacitor_SMD:C_0603_1608Metric, symbol Device:C_Small
- Q2: Height (mm) (none) -> 1.10; Height(mm) 1.1mm -> (none)
- QD1, QD2, QD3, QD4, QD5, QD6, QD7, QD8: Characteristics (none) -> MOSFET N Ch 60Vds, +- 20Vgs, 380mA, 2.5Ohms, 420mW, AEC-Q10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; Height (mm) (none) -> 1.10; MFN (none) -> onsemi; MFP (none) -> 2V7002KT1G; Mouser Part Number (none) -> 863-2V7002KT1G; Mouser Price/Stock (none) -> https://www.mouser.com/ProductDetail/onsemi/2V7002KT1G?qs=3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; Package (none) -> SOT-23-3; Type (none) -> SMD
- RP1, RP2, RP3, RP4, RP5, RP6, RP7, RP8: symbol Device:R_Small -> Device:R; Characteristics Thick Film Resistor - 10KΩ 5% 300mW; Anti Surge AEC-Q200; 1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 -> Thick Film Resistors - SMD 0603 10Kohm 5% Anti Surge AEC-Q2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
Connections:
- net GNDPWR: now also C11.2
- net VSYS: now also C11.1
- net PG: now reaches U1.30 (RUN)
- no-connect marks 25 -> 24
Other:
- moved on the sheet: RP1, RP2, RP3, RP4, RP5, RP6, RP7, RP8

Commit message: Pre KiCad 7.0.0 WIP
Parts:
- QD1, QD2, QD3, QD4, QD5, QD6, QD7, QD8: footprint Package_TO_SOT_SMD:SOT-23 -> dragon_mobile:2V7002KT1G
Connections:
- net BANK_A.CNTL1 renamed BANK_A.OUT1
- net BANK_A.CNTL2 renamed BANK_A.OUT2
- net BANK_A.CNTL3 renamed BANK_A.OUT3
- net BANK_A.CNTL4 renamed BANK_A.OUT4
- net BANK_B.CNTL5 renamed BANK_B.OUT5
- net BANK_B.CNTL6 renamed BANK_B.OUT6
- net BANK_B.CNTL7 renamed BANK_B.OUT7
- net BANK_B.CNTL8 renamed BANK_B.OUT8
Changed lines of the file:
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@@
     (effects (font (size 1.27 1.27)) (justify left bottom))
   )
-  (label "BANK_A.CNTL1" (at 167.64 48.26 180)
+  (label "BANK_A.OUT1" (at 167.64 48.26 180)
     (effects (font (size 1.27 1.27)) (justify right bottom))
   )
-  (label "BANK_A.CNTL2" (at 167.64 63.5 180)
+  (label "BANK_A.OUT2" (at 167.64 63.5 180)
     (effects (font (size 1.27 1.27)) (justify right bottom))
   )
@@
     (effects (font (size 1.27 1.27)) (justify left bottom))
   )
-  (label "BANK_B.CNTL7" (at 167.64 139.7 180)
+  (label "BANK_B.OUT7" (at 167.64 139.7 180)
     (effects (font (size 1.27 1.27)) (justify right bottom))
   )
-  (label "BANK_A.CNTL3" (at 167.64 78.74 180)
+  (label "BANK_A.OUT3" (at 167.64 78.74 180)
     (effects (font (size 1.27 1.27)) (justify right bottom))
   )
@@
     (effects (font (size 1.27 1.27)) (justify left bottom))
   )
-  (label "BANK_B.CNTL6" (at 167.64 124.46 180)
+  (label "BANK_B.OUT6" (at 167.64 124.46 180)
     (effects (font (size 1.27 1.27)) (justify right bottom))
   )
@@
     (effects (font (size 1.27 1.27)) (justify left bottom))
   )
-  (label "BANK_B.CNTL5" (at 167.64 109.22 180)
+  (label "BANK_B.OUT5" (at 167.64 109.22 180)
     (effects (font (size 1.27 1.27)) (justify right bottom))
   )
-  (label "BANK_B.CNTL8" (at 167.64 154.94 180)
+  (label "BANK_B.OUT8" (at 167.64 154.94 180)
     (effects (font (size 1.27 1.27)) (justify right bottom))
   )
@@
     (effects (font (size 1.27 1.27)) (justify left bottom))
   )
-  (label "BANK_A.CNTL4" (at 167.64 93.98 180)
+  (label "BANK_A.OUT4" (at 167.64 93.98 180)
     (effects (font (size 1.27 1.27)) (justify right bottom))
   )
@@
     (effects (font (size 1.27 1.27)) (justify left bottom))
   )
-  (hierarchical_label "BANK_A{CNTL[1..4]}" (shape output) (at 203.2 43.18 0)
+  (hierarchical_label "BANK_A{OUT[1..4]}" (shape output) (at 203.2 43.18 0)
     (effects (font (size 2 2) (thickness 0.4) bold) (justify left))
   )
@@
     (effects (font (size 2 2) bold) (justify right))
   )
-  (hierarchical_label "BANK_B{CNTL[5..8]}" (shape output) (at 203.2 104.14 0)
+  (hierarchical_label "BANK_B{OUT[5..8]}" (shape output) (at 203.2 104.14 0)
     (effects (font (size 2 2) (thickness 0.4) bold) (justify left))
   )
@@
       (effects (font (size 1.27 1.27)) (justify left) hide)
     )
-    (property "Footprint" "Package_TO_SOT_SMD:SOT-23" (id 2) (at 151.13 118.745 0)
+    (property "Footprint" "dragon_mobile:2V7002KT1G" (id 2) (at 151.13 118.745 0)
       (effects (font (size 1.27 1.27) italic) (justify left) hide)
     )
@@
       (effects (font (size 1.27 1.27)) (justify left) hide)
     )
-    (property "Footprint" "Package_TO_SOT_SMD:SOT-23" (id 2) (at 151.13 88.265 0)
+    (property "Footprint" "dragon_mobile:2V7002KT1G" (id 2) (at 151.13 88.265 0)
       (effects (font (size 1.27 1.27) italic) (justify left) hide)
     )
@@
       (effects (font (size 1.27 1.27)) (justify left) hide)
     )
-    (property "Footprint" "Package_TO_SOT_SMD:SOT-23" (id 2) (at 151.13 179.705 0)
+    (property "Footprint" "dragon_mobile:2V7002KT1G" (id 2) (at 151.13 179.705 0)
       (effects (font (size 1.27 1.27) italic) (justify left) hide)
     )
@@
       (effects (font (size 1.27 1.27)) (justify left) hide)
     )
-    (property "Footprint" "Package_TO_SOT_SMD:SOT-23" (id 2) (at 151.13 103.505 0)
+    (property "Footprint" "dragon_mobile:2V7002KT1G" (id 2) (at 151.13 103.505 0)
       (effects (font (size 1.27 1.27) italic) (justify left) hide)
     )
@@
       (effects (font (size 1.27 1.27)) (justify left) hide)
     )
-    (property "Footprint" "Package_TO_SOT_SMD:SOT-23" (id 2) (at 151.13 164.465 0)
+    (property "Footprint" "dragon_mobile:2V7002KT1G" (id 2) (at 151.13 164.465 0)
       (effects (font (size 1.27 1.27) italic) (justify left) hide)
     )
@@
       (effects (font (size 1.27 1.27)) (justify left) hide)
     )
-    (property "Footprint" "Package_TO_SOT_SMD:SOT-23" (id 2) (at 151.13 149.225 0)
+    (property "Footprint" "dragon_mobile:2V7002KT1G" (id 2) (at 151.13 149.225 0)
       (effects (font (size 1.27 1.27) italic) (justify left) hide)
     )
@@
       (effects (font (size 1.27 1.27)) (justify left) hide)
     )
-    (property "Footprint" "Package_TO_SOT_SMD:SOT-23" (id 2) (at 151.13 73.025 0)
+    (property "Footprint" "dragon_mobile:2V7002KT1G" (id 2) (at 151.13 73.025 0)
       (effects (font (size 1.27 1.27)) (justify left) hide)
     )
@@
       (effects (font (size 1.27 1.27)) (justify left) hide)
     )
-    (property "Footprint" "Package_TO_SOT_SMD:SOT-23" (id 2) (at 151.13 133.985 0)
+    (property "Footprint" "dragon_mobile:2V7002KT1G" (id 2) (at 151.13 133.985 0)
       (effects (font (size 1.27 1.27) italic) (justify left) hide)
     )

Commit message: Commit before removing git submodule
Parts:
- renumbered C11 to C12
Connections:
- net +5V: now also C12.1
- net IO1: now also U1.10 (GPIO7); no longer U1.6 (GPIO4)
- net IO2: now also U1.9 (GPIO6); no longer U1.5 (GPIO3)
- net IO3: now also U1.7 (GPIO5); no longer U1.4 (GPIO2)
- net IO4: now also U1.6 (GPIO4); no longer U1.2 (GPIO1)
- net IO5: now also U1.1 (GPIO0); no longer U1.11 (GPIO8)
- net IO6: now also U1.2 (GPIO1); no longer U1.10 (GPIO7)
- net IO7: now also U1.4 (GPIO2); no longer U1.9 (GPIO6)
- net IO8: now also U1.5 (GPIO3); no longer U1.7 (GPIO5)
- net VSYS: no longer C12.1
Other:
- note added: "${SHEETNAME}"
- note removed: "PicoW Control / Drivers"
- company: (none) -> Michael Cummings
- title: (none) -> Pico W SSR Control
- moved on the sheet: C12, Q2
