File: hardware/picow_ssr_control/picow_ssr_control.kicad_pcb (KiCad board)
At the start: 2 copper layers, 65 x 90 mm, 65 parts, among them Q1 SQ3419EV-T1_GE3, Q2 DMG2305UX-7, U1 RaspberryPi-PicoW, U2 LMR33610BDDAR

Commit message: Pre KiCad 7.0.0 WIP
Parts:
- QD1, QD2, QD3, QD4, QD5, QD6, QD7, QD8: footprint Package_TO_SOT_SMD:SOT-23 -> dragon_mobile:2V7002KT1G
- moved FID3 10.0 mm to (76.5, 91.0)
- moved H2 10.0 mm to (21.5, 91.0)
- moved S1 9.73 mm to (60.7, 88.7)
- moved REF_KiCAD 9.09 mm to (60.7, 88.0)
- moved OSHW_Mono_0.1_Scale 6.97 mm to (36.0, 89.8)
- moved RP8 6.39 mm to (42.5, 70.1)
- moved RP5 6.35 mm to (42.5, 79.8)
- moved RP7 6.29 mm to (42.5, 73.3)
- moved RP6 6.28 mm to (42.5, 76.6)
- moved JS1 5.02 mm to (72.4, 40.5)
- moved JS2 5.02 mm to (71.4, 37.8)
- moved JCNTL1 5.02 mm to (74.3, 45.5)
- moved JCNTL2 5.02 mm to (74.3, 66.5)
- moved FID2 5.00 mm to (76.5, 23.5)
- moved H3 5.00 mm to (76.5, 56.0)
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Connections:
- net /Control Out/BANK_A.CNTL1 renamed /Control Out/BANK_A.OUT1
- net /Control Out/BANK_A.CNTL2 renamed /Control Out/BANK_A.OUT2
- net /Control Out/BANK_A.CNTL3 renamed /Control Out/BANK_A.OUT3
- net /Control Out/BANK_A.CNTL4 renamed /Control Out/BANK_A.OUT4
- net /Control Out/BANK_B.CNTL5 renamed /Control Out/BANK_B.OUT5
- net /Control Out/BANK_B.CNTL6 renamed /Control Out/BANK_B.OUT6
- net /Control Out/BANK_B.CNTL7 renamed /Control Out/BANK_B.OUT7
- net /Control Out/BANK_B.CNTL8 renamed /Control Out/BANK_B.OUT8
- net /Control Out/a1o renamed /Control Out/OUT1
- net /Control Out/a2o renamed /Control Out/OUT2
- net /Control Out/a3o renamed /Control Out/OUT3
- net /Control Out/a4o renamed /Control Out/OUT4
- net /Control Out/a5o renamed /Control Out/OUT5
- net /Control Out/a6o renamed /Control Out/OUT6
- net /Control Out/a7o renamed /Control Out/OUT7
- net /Control Out/a8o renamed /Control Out/OUT8
Routing:
- net /Control Out/BANK_B.OUT8: track 40.3 -> 34.0 mm
- net /Pico W Control/PG: track 60.7 -> 66.0 mm
- net /Control Out/BANK_B.OUT7: track 36.3 -> 31.2 mm
- net /Control Out/BANK_A.OUT4: track 42.4 -> 38.0 mm
- net /Control Out/BANK_B.OUT6: track 32.3 -> 28.5 mm
- net /Control Out/BANK_A.OUT3: track 46.4 -> 42.7 mm
- net /Pico W Control/IO8: track 30.2 -> 33.8 mm
- net /Control Out/BANK_A.OUT1: track 54.4 -> 51.0 mm
- net /Control Out/BANK_A.OUT2: track 50.4 -> 47.0 mm
- net /Pico W Control/IO7: track 40.1 -> 43.1 mm
- net +BATT: track 7.23 -> 4.44 mm, vias 6 -> 17
- net /Control Out/BANK_B.OUT5: track 28.2 -> 25.5 mm
- net +5V: track 93.5 -> 90.8 mm
- net /Pico W Control/IO6: track 47.6 -> 49.7 mm
- net /Pico W Control/IO1: track 12.8 -> 14.7 mm
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Other:
- board size 65 x 90 mm -> 65 x 80 mm
- board text added: "+BATT OUT1 OUT2 OUT3 OUT4"
- board text added: "0"
- board text added: "0 mm"
- board text added: "0.01 mm"
- board text added: "0.02"
- board text added: "0.035 mm"
- board text added: "1"
- board text added: "1 mm"
- board text added: "1.0900 mm"
- board text added: "3.3"
- board text added: "4.5"
- board text added: "65.0000 mm x 80.0000 mm"
- board text added: "B.Cu"
- board text added: "B.Mask"
- board text added: "B.Paste"
- board text added: "B.Silkscreen"
- board text added: "Bottom Silk Screen"
- board text added: "Bottom Solder Mask"
- board text added: "Bottom Solder Paste"
- board text added: "Color"
- board text added: "Dielectric 1"
- board text added: "Epsilon R"
- board text added: "F.Cu"
- board text added: "F.Mask"
- board text added: "F.Paste"
- board text added: "F.Silkscreen"
- board text added: "FR4"
- board text added: "Green"
- board text added: "Layer Name"
- board text added: "Loss Tangent"
- board text added: "Material"
- board text added: "Not specified"
- board text added: "OUT8 OUT7 OUT6 OUT5 +BATT"
- board text added: "Thickness (mm)"
- board text added: "Top Silk Screen"
- board text added: "Top Solder Mask"
- board text added: "Top Solder Paste"
- board text added: "Type"
- board text added: "White"
- board text added: "copper"
- board text added: "core"
- board text removed: "+BATT CNTL1 CNTL2 CNTL3 CNTL4"
- board text removed: "1.1600 mm"
- board text removed: "65.0000 mm x 90.0000 mm"
- board text removed: "CNTL8 CNTL7 CNTL6 CNTL5 +BATT"

Commit message: Commit before trying changes to power system
Parts:
- added JCNTL1_Label: JCNTL1_Label, dragon_mobile:JCNTL1_Label, F.Cu at (76.0, 36.8)
- added JCNTL2_Label: JCNTL2_Label, dragon_mobile:JCNTL2_Label, F.Cu at (76.0, 83.5)
- moved OSHW_Mono_0.1_Scale 6.50 mm to (42.5, 90.0)
Other:
- board text added: "v0.0.12"
- board text removed: "+"
- board text removed: "+BATT OUT1 OUT2 OUT3 OUT4"
- board text removed: "OUT8 OUT7 OUT6 OUT5 +BATT"
- board text removed: "v0.0.11"

Commit message: Commit before removing git submodule
Parts:
- removed JCNTL1, JCNTL2: SHF-105-01-L-D-RA, dragon_mobile:SAMTEC_SHF-105-01-L-D-RA
- removed JS1: SolderJumper_3_Bridged12, Jumper:SolderJumper-3_P1.3mm_Bridged12_RoundedPad1.0x1.5mm_NumberLabels
- removed JS2: Conn_01x02, dragon_mobile:PinHeader_1x02_P1.00mm_Vertical
- removed QRCode1: GitHub URL, LOGO
- added C12: 100n, Capacitor_SMD:C_0603_1608Metric, F.Cu at (23.3, 61.5)
- added JCTL1: SHF-105-01-L-D-RA, dragon_mobile:SAMTEC_SHF-105-01-L-D-RA, F.Cu at (74.3, 45.5)
- added JCTL2: SHF-105-01-L-D-RA, dragon_mobile:SAMTEC_SHF-105-01-L-D-RA, F.Cu at (74.3, 66.5)
- added JL2: Conn_01x02, dragon_mobile:PinHeader_1x02_P1.00mm_Vertical, F.Cu at (21.0, 38.7)
- added JP2: SolderJumper_2_Open, Jumper:SolderJumper-2_P1.3mm_Open_RoundedPad1.0x1.5mm, B.Cu at (73.0, 74.5)
- added JP3: Conn_01x02, dragon_mobile:PinHeader_1x02_P1.00mm_Vertical, F.Cu at (69.6, 34.7)
- C11: value 100n -> 4u7; footprint Capacitor_SMD:C_0603_1608Metric -> Capacitor_SMD:C_0805_2012Metric
- C3: value 220n -> 4u7; footprint Capacitor_SMD:C_0603_1608Metric -> Capacitor_SMD:C_0805_2012Metric
- C4: value 1u -> 220n
- C5: value 100n -> 1u
- C6: value 4u7 -> 100n; footprint Capacitor_SMD:C_0805_2012Metric -> Capacitor_SMD:C_0603_1608Metric
- JL1: value Conn_01x02 -> SolderJumper_2_Bridged; footprint dragon_mobile:PinHeader_1x02_P1.00mm_Vertical -> Jumper:SolderJumper-2_P1.3mm_Bridged_RoundedPad1.0x1.5mm
- JP1: moved to B.Cu
- OSHW_Mono_0.1_Scale: value US002122 -> ${COMMENT5}
- moved FID2 83.3 mm to (21.5, 86.0)
- moved JL1 55.5 mm to (20.0, 45.5)
- moved RL1 54.8 mm to (20.0, 41.8), turned to 90 degrees
- moved LP1 54.7 mm to (20.8, 36.1)
- moved C11 37.8 mm to (52.3, 36.7), turned to 0 degrees
- moved C6 18.6 mm to (53.9, 21.0), turned to -90 degrees
- moved R1 13.7 mm to (60.9, 32.4)
- moved ZD1 12.5 mm to (60.9, 36.1), turned to 90 degrees
- moved RP8 11.5 mm to (49.7, 61.1)
- moved JP1 11.4 mm to (73.0, 35.7), turned to 180 degrees
- moved C1 11.2 mm to (56.4, 37.0), turned to 180 degrees
- moved C7 11.0 mm to (52.3, 26.8)
- moved RP7 10.9 mm to (49.7, 65.1)
- moved C4 10.7 mm to (56.6, 29.9), turned to 180 degrees
- moved RP6 10.4 mm to (49.7, 69.1)
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Connections:
- net Net-(Q1-Pad3) renamed /Power Management/ZD
- C11 pad 1: /Pico W Control/VSYS -> +5V
- C4 pad 1: /Power Management/VCC -> /Power Management/VDC
- C5 pad 1: /Power Management/BOOT -> /Power Management/VCC
- C5 pad 2: /Power Management/SW -> GNDPWR
- C6 pad 1: +5V -> /Power Management/BOOT
- C6 pad 2: GNDPWR -> /Power Management/SW
- JL1 pad 1: GNDPWR -> +5V
- JL1 pad 2: Net-(JL1-Pad2) -> Net-(JL1-B)
- JP1 pad 1: +5V -> /Control Out/PI1
- JP1 pad 2: Net-(JP1-Pad2) -> +BATT
- LP1 pad 2: Net-(JL1-Pad2) -> Net-(JL2-Pin_2)
- RL1 pad 1: Net-(JP1-Pad2) -> Net-(JL1-B)
- RL1 pad 2: Net-(JL1-Pad2) -> Net-(JL2-Pin_2)
- U1 pad 1: unconnected-(U1-Pad1) -> /Pico W Control/IO5
- U1 pad 10: /Pico W Control/IO6 -> /Pico W Control/IO1
- U1 pad 11: /Pico W Control/IO5 -> unconnected-(U1-GPIO8-Pad11)
- U1 pad 2: /Pico W Control/IO4 -> /Pico W Control/IO6
- U1 pad 4: /Pico W Control/IO3 -> /Pico W Control/IO7
- U1 pad 5: /Pico W Control/IO2 -> /Pico W Control/IO8
- U1 pad 6: /Pico W Control/IO1 -> /Pico W Control/IO4
- U1 pad 7: /Pico W Control/IO8 -> /Pico W Control/IO3
- U1 pad 9: /Pico W Control/IO7 -> /Pico W Control/IO2
Routing:
- net /Pico W Control/IO5: track 56.3 -> 10.5 mm
- net +BATT: track 4.44 -> 45.4 mm
- net /Pico W Control/IO6: track 49.7 -> 9.79 mm
- net /Pico W Control/IO7: track 43.1 -> 10.1 mm
- net /Control Out/PwrIn2: track 30.1 -> 0.00 mm
- net /Pico W Control/IO8: track 33.8 -> 8.62 mm
- net /Control Out/BANK_A.OUT4: track 38.0 -> 53.7 mm
- net /Control Out/BANK_A.OUT3: track 42.7 -> 56.2 mm
- net /Power Management/VCC: track 3.83 -> 15.0 mm, vias 0 -> 2
- net /Control Out/BANK_B.OUT6: track 28.5 -> 37.6 mm
- net /Control Out/BANK_B.OUT5: track 25.5 -> 33.6 mm
- net /Control Out/BANK_B.OUT8: track 34.0 -> 41.9 mm
- net /Pico W Control/IO1: track 14.7 -> 7.07 mm
- net /Control Out/PI1: track 0.00 -> 7.30 mm
- net /Pico W Control/IO2: track 13.2 -> 6.46 mm
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Other:
- board text added: "+5V"
- board text added: "1.6 mm"
- board text added: "1.6900 mm"
- board text added: "Blue"
- board text added: "Liquid Ink"
- board text added: "Manual Control"
- board text added: "O1"
- board text added: "O2"
- board text added: "O3"
- board text added: "O4"
- board text added: "O5"
- board text added: "O6"
- board text added: "O7"
- board text added: "O8"
- board text added: "ON"
- board text added: "https://github.com/dragon-mobile/picow_ssr_control"
- board text added: "v${REVISION}"
- board text added: "© 2023 ${COMPANY}"
- board text removed: "1 mm"
- board text removed: "1.0900 mm"
- board text removed: "A1"
- board text removed: "A2"
- board text removed: "A3"
- board text removed: "A4"
- board text removed: "B5"
- board text removed: "B6"
- board text removed: "B7"
- board text removed: "B8"
- board text removed: "Green"
- board text removed: "v0.0.12"
- board text removed: "© 2023 Michael Cummings"
