File: hardware/picow_ssr_control/picow_ssr_control.kicad_sch (KiCad schematic)
At the start: 6 parts

Commit message: Commit before removing git submodule
Other:
- sheet Control Out ports: added PI[1..2]; removed +BATT
- sheet Power Management ports: added PI[1..2]; removed +BATT
- note added: "${TITLE}"
- note removed: "Pico W SSR Control"
- company: (none) -> Michael Cummings
- title: Picow SSR Control -> Pico W SSR Control
Changed lines of the file:
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@@
   (paper "USLetter")
   (title_block
-    (title "Picow SSR Control")
-    (date "2023-02-13")
-    (rev "0.0.11")
-    (comment 2 "http://creativecommons.org/licenses/by-sa/4.0/")
-    (comment 3 "License: CC By SA 4.0")
-    (comment 4 "Author: Michael Cummings")
-    (comment 5 "https://ohwr.org/project/cernohl/wikis/Documents/CERN-OHL-version-2")
-    (comment 6 "Hardware License: CERN-OHL-W")
+    (title "Pico W SSR Control")
+    (date "2023-03-14")
+    (rev "0.0.12")
+    (company "Michael Cummings")
+    (comment 1 "https://ohwr.org/project/cernohl/wikis/Documents/CERN-OHL-version-2")
+    (comment 2 "Hardware License: CERN-OHL-W")
+    (comment 3 "https://creativecommons.org/licenses/by-sa/4.0/")
+    (comment 4 "License: CC By SA 4.0")
   )
   (junction (at 111.76 45.72) (diameter 0) (color 255 255 0 1)
@@
   )
   (polyline (pts (xy 63.5 129.54) (xy 63.5 200.66))
-    (stroke (width 0) (type default))
-  )
-  (wire (pts (xy 124.46 27.94) (xy 124.46 40.64))
     (stroke (width 0) (type default))
   )
@@
     (stroke (width 0) (type default))
   )
+  (bus (pts (xy 127 40.64) (xy 132.08 40.64))
+    (stroke (width 0) (type default))
+  )
   (polyline (pts (xy 17.78 172.72) (xy 40.64 172.72))
     (stroke (width 0) (type default))
@@
     (stroke (width 0) (type default) (color 255 255 0 1))
   )
+  (bus (pts (xy 50.8 25.4) (xy 127 25.4))
+    (stroke (width 0) (type default))
+  )
   (polyline (pts (xy 45.72 137.16) (xy 45.72 167.64))
     (stroke (width 0) (type default))
@@
     (stroke (width 0) (type default))
   )
-  (wire (pts (xy 124.46 40.64) (xy 132.08 40.64))
-    (stroke (width 0) (type default))
-  )
   (wire (pts (xy 45.72 45.72) (xy 60.96 45.72))
+    (stroke (width 0) (type default))
+  )
+  (bus (pts (xy 127 25.4) (xy 127 40.64))
     (stroke (width 0) (type default))
   )
@@
     (stroke (width 0) (type default) (color 255 255 0 1))
   )
+  (bus (pts (xy 45.72 40.64) (xy 50.8 40.64))
+    (stroke (width 0) (type default))
+  )
   (polyline (pts (xy 40.64 195.58) (xy 17.78 195.58))
-    (stroke (width 0) (type default))
-  )
-  (wire (pts (xy 50.8 27.94) (xy 124.46 27.94))
     (stroke (width 0) (type default))
   )
@@
     (stroke (width 0) (type default) (color 255 255 0 1))
   )
-  (wire (pts (xy 45.72 40.64) (xy 50.8 40.64))
-    (stroke (width 0) (type default))
-  )
   (bus (pts (xy 99.06 45.72) (xy 111.76 45.72))
     (stroke (width 0) (type default) (color 255 255 0 1))
@@
     (stroke (width 0) (type default))
   )
-  (wire (pts (xy 50.8 40.64) (xy 50.8 27.94))
+  (bus (pts (xy 50.8 40.64) (xy 50.8 25.4))
     (stroke (width 0) (type default))
   )
@@
     )
   )
-  (text "Pico W SSR Control" (at 15.24 20.32 0)
+  (text "${TITLE}" (at 15.24 20.32 0)
     (effects (font (size 4 4) bold) (justify left bottom))
   )
@@
     )
   )
+  (symbol (lib_name "Fiducial_2") (lib_id "Mechanical:Fiducial") (at 25.4 185.42 0) (unit 1)
+    (in_bom no) (on_board yes) (dnp no) (fields_autoplaced)
+    (property "Reference" "FID2" (at 27.686 185.4199 0)
+      (effects (font (size 1.27 1.27)) (justify left))
+    )
+    (property "Value" "Fiducial" (at 27.94 186.6899 0)
+      (effects (font (size 1.27 1.27)) (justify left) hide)
+    )
+    (property "Footprint" "Fiducial:Fiducial_0.5mm_Mask1mm" (at 25.4 185.42 0)
+      (effects (font (size 1.27 1.27)) hide)
+    )
+    (property "Datasheet" "~" (at 25.4 185.42 0)
+      (effects (font (size 1.27 1.27)) hide)
+    )
+    (instances
+      (project "picow_ssr_control"
+        (path "/04b3a773-2568-4dd5-b3b9-f3130861ac39"
+          (reference "FID2") (unit 1)
+        )
+      )
+    )
+  )
+  (symbol (lib_id "Mechanical:MountingHole_Pad") (at 30.48 152.4 270) (unit 1)
+    (in_bom no) (on_board yes) (dnp no) (fields_autoplaced)
+    (property "Reference" "H2" (at 34.29 151.1299 90)
+      (effects (font (size 1.27 1.27)) (justify left))
+    )
+    (property "Value" "MountingHole_Pad" (at 34.29 153.6699 90)
+      (effects (font (size 1.27 1.27)) (justify left) hide)
+    )
+    (property "Footprint" "MountingHole:MountingHole_3.2mm_M3_Pad_Via" (at 30.48 152.4 0)
+      (effects (font (size 1.27 1.27)) hide)
+    )
+    (property "Datasheet" "~" (at 30.48 152.4 0)
+      (effects (font (size 1.27 1.27)) hide)
+    )
+    (pin "1")
+    (instances
+      (project "picow_ssr_control"
+        (path "/04b3a773-2568-4dd5-b3b9-f3130861ac39"
+          (reference "H2") (unit 1)
+        )
+      )
+    )
+  )
   (symbol (lib_id "power:GNDPWR") (at 27.94 162.56 0) (unit 1)
     (in_bom yes) (on_board yes) (dnp no)
@@
       (effects (font (size 1.27 1.27)) hide)
     )
-    (property "Value" "GNDPWR" (at 27.94 165.862 0)
+    (property "Value" "GNDPWR" (at 27.94 166.116 0)
       (effects (font (size 1.27 1.27)))
     )
@@
     )
   )
-  (symbol (lib_name "Fiducial_2") (lib_id "Mechanical:Fiducial") (at 25.4 185.42 0) (unit 1)
-    (in_bom no) (on_board yes) (dnp no) (fields_autoplaced)
-    (property "Reference" "FID2" (at 27.686 185.4199 0)
-      (effects (font (size 1.27 1.27)) (justify left))
-    )
-    (property "Value" "Fiducial" (at 27.94 186.6899 0)
-      (effects (font (size 1.27 1.27)) (justify left) hide)
-    )
-    (property "Footprint" "Fiducial:Fiducial_0.5mm_Mask1mm" (at 25.4 185.42 0)
-      (effects (font (size 1.27 1.27)) hide)
-    )
-    (property "Datasheet" "~" (at 25.4 185.42 0)
-      (effects (font (size 1.27 1.27)) hide)
-    )
-    (instances
-      (project "picow_ssr_control"
-        (path "/04b3a773-2568-4dd5-b3b9-f3130861ac39"
-          (reference "FID2") (unit 1)
-        )
-      )
-    )
-  )
-  (symbol (lib_id "Mechanical:MountingHole_Pad") (at 30.48 152.4 270) (unit 1)
-    (in_bom no) (on_board yes) (dnp no) (fields_autoplaced)
-    (property "Reference" "H2" (at 34.29 151.1299 90)
-      (effects (font (size 1.27 1.27)) (justify left))
-    )
-    (property "Value" "MountingHole_Pad" (at 34.29 153.6699 90)
-      (effects (font (size 1.27 1.27)) (justify left) hide)
-    )
-    (property "Footprint" "MountingHole:MountingHole_3.2mm_M3_Pad_Via" (at 30.48 152.4 0)
-      (effects (font (size 1.27 1.27)) hide)
-    )
-    (property "Datasheet" "~" (at 30.48 152.4 0)
-      (effects (font (size 1.27 1.27)) hide)
-    )
-    (pin "1")
-    (instances
-      (project "picow_ssr_control"
-        (path "/04b3a773-2568-4dd5-b3b9-f3130861ac39"
-          (reference "H2") (unit 1)
-        )
-      )
-    )
-  )
   (symbol (lib_id "Mechanical:Fiducial") (at 25.4 180.34 0) (unit 1)
     (in_bom no) (on_board yes) (dnp no) (fields_autoplaced)
@@
       (effects (font (size 1.27 1.27)) (justify left))
     )
-    (pin "+BATT" output (at 132.08 40.64 180)
+    (pin "PI[1..2]" output (at 132.08 40.64 180)
       (effects (font (size 1.27 1.27)) (justify left))
     )
@@
       (effects (font (size 1.27 1.27)) (justify right))
     )
-    (pin "+BATT" input (at 45.72 40.64 0)
+    (pin "PI[1..2]" input (at 45.72 40.64 0)
       (effects (font (size 1.27 1.27)) (justify right))
     )
